File: HWmonitor_DSPlink.kicad_pcb (KiCad board)
At the start: 2 copper layers, 56 x 66 mm, 100 parts, among them J1 Mini USB-B, J2 IDC-Header 2x4, T1 760390014, U1 FT232RL, U10 OPA197xDBV, U11 OPA197xDBV, U12 USBLC6-2SC6, U2 ISO7830DWW, U3 ISO7821DWW, U4 SN6501DBVR, U5 TL431BCDBZ, U6 AD5324ARMZ, U7 TLV70450DBVT, U8 OPA197xDBV, U9 OPA197xDBV, X1 Conn_Coaxial, X2 Conn_Coaxial, X3 Conn_Coaxial, X4 Conn_Coaxial

Commit message: BOM bug, LED resistor to 270R
Parts:
- R4: value 10R -> 270R
